File: ROORRR/ROORRR.sch (KiCad schematic (older format))
At the start: 88 parts, among them SW1 SW_Push, U1 ATmega32U4-AU, Y1 16MHz

Commit message: checkpoint 1
Parts:
- removed USB1: Molex-0548190589, random-keyboard-parts:Molex-0548190589, symbol random-keyboard-parts:Molex-0548190589
- added J1: AVR-ISP-6, random-keyboard-parts:Reset_Pretty-Mask, symbol Connector:AVR-ISP-6
- added R5, R6: 5.1k, Resistor_SMD:R_0805_2012Metric_Pad1.15x1.40mm_HandSolder, symbol Device:R_Small
- added U2: PRTR5V0U2X, random-keyboard-parts:SOT143B, symbol random-keyboard-parts:PRTR5V0U2X
- added USB1: HRO-TYPE-C-31-M-12, Type-C:HRO-TYPE-C-31-M-12-HandSoldering, symbol Type-C:HRO-TYPE-C-31-M-12
- C1, C2, C3, C4, C5, C6, C7: footprint Capacitor_SMD:C_0805_2012Metric -> Capacitor_SMD:C_0805_2012Metric_Pad1.15x1.40mm_HandSolder
- F1: footprint Fuse:Fuse_1206_3216Metric -> Fuse:Fuse_1206_3216Metric_Pad1.42x1.75mm_HandSolder
- MX1: value MX-NoLED -> Q
- MX11: value MX-NoLED -> A
- MX12: value MX-NoLED -> S
- MX13: value MX-NoLED -> D
- MX14: value MX-NoLED -> F
- MX15: value MX-NoLED -> G
- MX16: value MX-NoLED -> H
- MX17: value MX-NoLED -> J
- MX18: value MX-NoLED -> K
- MX19: value MX-NoLED -> L
- MX2: value MX-NoLED -> W
- MX21: value MX-NoLED -> Z
- MX22: value MX-NoLED -> X
- MX23: value MX-NoLED -> C
- MX24: value MX-NoLED -> V
- MX25: value MX-NoLED -> B
- MX26: value MX-NoLED -> N
- MX27: value MX-NoLED -> M
- MX28: value MX-NoLED -> ,
- MX29: value MX-NoLED -> .
- MX3: value MX-NoLED -> E
- MX31: value MX-NoLED -> 1
- MX32: value MX-NoLED -> 2
- MX33: value MX-NoLED -> 3
- MX34: value MX-NoLED -> 4
- MX35: value MX-NoLED -> 5
- MX36: value MX-NoLED -> 6
- MX37: value MX-NoLED -> 7
- MX38: value MX-NoLED -> 8
- MX39: value MX-NoLED -> 9
- MX4: value MX-NoLED -> R
- MX5: value MX-NoLED -> T
- MX6: value MX-NoLED -> Y
- MX7: value MX-NoLED -> U
- MX8: value MX-NoLED -> I
- MX9: value MX-NoLED -> O
- R1, R2, R3, R4: footprint Resistor_SMD:R_0805_2012Metric -> Resistor_SMD:R_0805_2012Metric_Pad1.15x1.40mm_HandSolder
- Y1: footprint Crystal:Crystal_SMD_3225-4Pin_3.2x2.5mm -> Crystal:Crystal_SMD_3225-4Pin_3.2x2.5mm_HandSoldering
Connections:
- net labels added: DN, DP, MISO, MOSI, RESET, SCK
- wire segments 231 -> 258
- no-connect marks 0 -> 2

Commit message: checkpoint 2
Parts:
- removed C4: 0.1uF, Capacitor_SMD:C_0805_2012Metric_Pad1.15x1.40mm_HandSolder, symbol Device:C_Small
- added C8: 0.1uF, Capacitor_SMD:C_0805_2012Metric_Pad1.15x1.40mm_HandSolder, symbol Device:C_Small
Connections:
- net labels added: XTAL1, XTAL2
- wire segments 258 -> 185
Other:
- moved on the sheet: C1, C2, C5, C6, C7, R1, SW1, Y1

Commit message: checkpoint2
Parts:
- USB1: footprint Type-C:HRO-TYPE-C-31-M-12-HandSoldering -> Type-C:HRO-TYPE-C-31-M-12
Changed lines of the file:
@@
 F 0 "USB1" H 4233 2197 60  0000 C CNN
 F 1 "HRO-TYPE-C-31-M-12" H 4233 2091 60  0000 C CNN
-F 2 "Type-C:HRO-TYPE-C-31-M-12-HandSoldering" H 4400 1400 60  0001 C CNN
+F 2 "Type-C:HRO-TYPE-C-31-M-12" H 4400 1400 60  0001 C CNN
 F 3 "" H 4400 1400 60  0001 C CNN
 	1    4400 1400
